File: pcb/mux_in-1b/mux_in-1b.kicad_pcb (KiCad board)
At the start: 2 copper layers, 34 x 61 mm, 56 parts, among them J1 Conn_01x16_Pin, J3 Conn_01x16_Pin, J4 Conn_01x02_Pin, J6 Conn_01x02_Pin, SW1 SW_DIP_x02, SW2 SW_Push

Commit message: Now with wifi, leds, and fixed integer overflow
Other:
- board text added: "R1"
- board text added: "R2"
Changed lines of the file:
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@@
+		)
+	)
+	(gr_text "R1"
+		(at 143.95 103.15 0)
+		(layer "F.SilkS")
+		(effects
+			(font
+				(size 1 1)
+				(thickness 0.1)
+			)
+			(justify left bottom)
+		)
+	)
+	(gr_text "R2"
+		(at 131.2 71.2 0)
+		(layer "F.SilkS")
+		(effects
+			(font
+				(size 1 1)
+				(thickness 0.1)
+			)
+			(justify left bottom)
 		)
 	)
@@
 		)
 	)
+	(gr_text "R2"
+		(at 153.4 108.6 180)
+		(layer "B.SilkS")
+		(effects
+			(font
+				(size 1 1)
+				(thickness 0.1)
+			)
+			(justify left bottom mirror)
+		)
+	)
+	(gr_text "G"
+		(at 158 114.8 0)
+		(layer "B.SilkS")
+		(effects
+			(font
+				(size 1 1)
+				(thickness 0.1)
+			)
+			(justify left bottom mirror)
+		)
+	)
+	(gr_text "G"
+		(at 137.6 121.6 0)
+		(layer "B.SilkS")
+		(effects
+			(font
+				(size 1 1)
+				(thickness 0.1)
+			)
+			(justify left bottom mirror)
+		)
+	)
+	(gr_text "VCC"
+		(at 158.8 107.6 0)
+		(layer "B.SilkS")
+		(effects
+			(font
+				(size 1 1)
+				(thickness 0.1)
+			)
+			(justify left bottom mirror)
+		)
+	)
+	(gr_text "VCC"
+		(at 137.6 116.4 90)
+		(layer "B.SilkS")
+		(effects
+			(font
+				(size 1 1)
+				(thickness 0.1)
+			)
+			(justify left bottom mirror)
+		)
+	)
+	(gr_text "R2"
+		(at 150.6 108.6 180)
+		(layer "B.SilkS")
+		(effects
+			(font
+				(size 1 1)
+				(thickness 0.1)
+			)
+			(justify left bottom mirror)
+		)
+	)
+	(gr_text "R2"
+		(at 150.2 73.8 180)
+		(layer "B.SilkS")
+		(effects
+			(font
+				(size 1 1)
+				(thickness 0.1)
+			)
+			(justify left bottom mirror)
+		)
+	)
