File: pcb/pico-control-2b/pico-control-2b.kicad_sch (KiCad schematic)
At the start: 26 parts, among them J1 Conn_01x07_Pin, J2 Conn_01x08_Socket, J4 Conn_01x02_Socket, SW1 SW_Push, SW2 SW_DIP_x02, U1 Pico

Commit message: PCB fixes and adjustments
Parts:
- added J5: Conn_01x02_Socket, Connector_PinHeader_2.54mm:PinHeader_1x02_P2.54mm_Vertical, symbol Connector:Conn_01x02_Socket
- added JP2: SolderJumper_2_Open, Jumper:SolderJumper-2_P1.3mm_Open_RoundedPad1.0x1.5mm, symbol Jumper:SolderJumper_2_Open
- added R5: R, digikey-footprints:1206, symbol Device:R
- J4: footprint digikey-footprints:PinHeader_1x2_P2.54mm -> Connector_PinHeader_2.54mm:PinHeader_1x02_P2.54mm_Vertical
Connections:
- net +5V: now also J5.2 (Pin_2)
- net GND: now also J5.1 (Pin_1)
- net at D4.1 (K), J2.1 (Pin_1), R1.2: now also JP2.1 (A), R5.2; no longer U1.31 (GPIO26_ADC0)
- new net: JP2.2 (B), R5.1, U1.31 (GPIO26_ADC0)
